Commit message: u

File: xacro/diffbot.xacro (robot description, xacro)
@@ -6,5 +6,5 @@
 <!-- *********************************************************************************************************************************  -->
 <!-- ****************************************************** Parameters ***************************************************************  -->
-  <xacro:property name="mesh_path"      value="package://robot_gazebo/meshes/diffbot/"/>
+  <xacro:property name="mesh_path"      value="package://diffbot/meshes/diffbot/"/>
   <xacro:property name="name_space"     value="diffbot"  />
   <xacro:property name="prefix"         value=""  />
@@ -36,6 +36,6 @@
   <xacro:property name="hokuyo_z"       value="${(hokuyo_height+base_height)/2}" />
 <!-- ****************************************************** Includes *****************************************************************  -->
-  <xacro:include filename="$(find robot_gazebo)/xacro/common_rviz_materials.xacro" />   <!-- RVIZ Colors                                -->
-  <xacro:include filename="$(find robot_gazebo)/gazebo/gz_diffbot.xacro" />             <!-- Gazebo                                     -->
+  <xacro:include filename="$(find diffbot)/xacro/common_rviz_materials.xacro" />   <!-- RVIZ Colors                                -->
+  <xacro:include filename="$(find diffbot)/gazebo/gz_diffbot.xacro" />             <!-- Gazebo                                     -->
 <!-- ****************************************************** Footprint ****************************************************************  -->
     <link name="${prefix}footprint"/>
