Commit message: u

File: gazebo/gz_diffbot.xacro (robot description, xacro)
@@ -14,124 +14,7 @@
     </gazebo>
 <!-- ******************************************************  Joint States Publisher **************************************************  -->
-  <gazebo>
-    <plugin name="joint_states_pub" filename="libgazebo_ros_joint_state_publisher.so">
-      <ros>
-        <namespace>${name_space}</namespace>
-      </ros>
-      <joint_name>${prefix}right_wheel_joint</joint_name>
-      <joint_name>${prefix}left_wheel_joint</joint_name>
-      <update_rate>100.0</update_rate>
-    </plugin>
- </gazebo>
 <!-- ******************************************************  Skid Steer Drive Controller *********************************************  -->
-  <gazebo>
-    <plugin name="skid_drive" filename="libgazebo_ros_diff_drive.so">
-      <ros>
-        <namespace>${name_space}</namespace>
-      </ros>
-      <num_wheel_pairs>1</num_wheel_pairs>
-      <!-- 1st Wheels Set -->
-      <right_joint>${prefix}right_wheel_joint</right_joint>
-      <left_joint>${prefix}left_wheel_joint</left_joint>
-      <wheel_separation>${wheel_y*2}</wheel_separation>
-      <wheel_diameter>${wheel_radius*2}</wheel_diameter>
-      <max_wheel_torque>20</max_wheel_torque>
-      <max_wheel_acceleration>1.0</max_wheel_acceleration>
-      <update_rate>100.0</update_rate>
-      <robot_base_frame>${prefix}footprint</robot_base_frame>
-      <odometry_frame>odom</odometry_frame>
-      <publish_odom>true</publish_odom>
-      <publish_odom_tf>true</publish_odom_tf>
-      <publish_wheel_tf>true</publish_wheel_tf>
-    </plugin>
-  </gazebo>
 <!-- ******************************************************  Camera ******************************************************************  -->
-  <gazebo reference="${prefix}camera">
-    <sensor type="camera" name="camera">
-      <update_rate>30.0</update_rate>
-      <camera name="head">
-        <horizontal_fov>${radians(80)}</horizontal_fov>
-        <image>
-          <width>1280</width>
-          <height>720</height>
-          <format>R8G8B8</format>
-        </image>
-        <clip>
-          <near>0.02</near>
-          <far>300</far>
-        </clip>
-        <noise>
-          <type>gaussian</type>
-          <!-- Noise is sampled independently per pixel on each frame.
-          That pixel's noise value is added to each of its color
-          channels, which at that point lie in the range [0,1]. -->
-          <mean>0.0</mean>
-          <stddev>0.007</stddev>
-        </noise>
-      </camera>
-      <plugin name="camera_controller" filename="libgazebo_ros_camera.so">
-        <ros>
-          <namespace>${name_space}</namespace>
-        </ros>
-        <alwaysOn>true</alwaysOn>
-        <updateRate>0.0</updateRate>
-        <cameraName>camera</cameraName>
-        <imageTopicName>image_raw</imageTopicName>
-        <cameraInfoTopicName>camera_info</cameraInfoTopicName>
-        <frameName>camera_optical</frameName>
-        <!-- setting hackBaseline to anything but 0.0 will cause a misalignment
-        between the gazebo sensor image and the frame it is supposed to
-        be attached to -->
-        <hackBaseline>0.0</hackBaseline>
-        <distortionK1>0.0</distortionK1>
-        <distortionK2>0.0</distortionK2>
-        <distortionK3>0.0</distortionK3>
-        <distortionT1>0.0</distortionT1>
-        <distortionT2>0.0</distortionT2>
-        <CxPrime>0</CxPrime>
-        <Cx>0.0</Cx>
-        <Cy>0.0</Cy>
-        <focalLength>0.0</focalLength>
-      </plugin>
-    </sensor>
-    <material>Gazebo/Green</material>
-  </gazebo>
 <!-- ****************************************************** hokuyo  ******************************************************************  -->
-  <gazebo reference="${prefix}hokuyo">
-    <sensor type="ray" name="head_hokuyo_sensor">
-      <plugin name="hokuyo" filename="libgazebo_ros_ray_sensor.so">
-        <ros>
-          <namespace>${name_space}</namespace>
-        </ros>
-        <output_type>sensor_msgs/LaserScan</output_type>
-      </plugin>
-      <update_rate>30</update_rate>
-      <pose>0 0 0 0 0 0</pose>
-      <visualize>false</visualize>
-      <ray>
-        <scan>
-          <horizontal>
-            <samples>720</samples>
-            <resolution>1</resolution>
-            <min_angle>-${radians(180)}</min_angle>
-            <max_angle> ${radians(180)}</max_angle>
-          </horizontal>
-        </scan>
-        <range>
-          <min>0.10</min>
-          <max>30.0</max>
-          <resolution>0.01</resolution>
-        </range>
-<!-- Noise parameters based on published spec for Hokuyo laser achieving "+-30mm" accuracy at range < 10m.  A mean of 0.0m and stddev   -->
-<!-- of 0.01m will put 99.7% of samples within 0.03m of the true reading.                                                               -->
-        <noise>
-          <type>gaussian</type>
-          <mean>0.0</mean>
-          <stddev>0.01</stddev>
-        </noise>
-      </ray>
-    </sensor>
-    <!-- <material>Gazebo/Red</material> -->
-  </gazebo>
 <!-- ****************************************************** END **********************************************************************  -->
 </robot>

File: xacro/diffbot.xacro (robot description, xacro)
@@ -222,5 +222,5 @@
       <origin xyz="0 0 0" rpy="0 0 0" />
       <geometry>
-        <mesh filename="${mesh_path}hokuyo.dae"/> <!--  <box size="${hokuyo_length} ${hokuyo_width} ${hokuyo_height}"/> -->
+        <box size="${hokuyo_length} ${hokuyo_width} ${hokuyo_height}"/>
       </geometry>
     </collision>
